File: Elétrica/glicosimetro/glicosimetro.kicad_sch (KiCad schematic)
At the start: 19 parts, among them U1 ESP32-C3_SUPERMINI, U2 MCP6L01Rx-xOT, U3 MCP6L01Rx-xOT, U4 LM1117DT-3.3, U5 MCP6L01Rx-xOT, U6 MCP6L01Rx-xOT, U7 MCP6L01Rx-xOT

Commit message: inicio da placa
Parts:
- removed R1, R2, R3: R, Resistor_SMD:R_0603_1608Metric_Pad0.98x0.95mm_HandSolder, symbol Device:R
- removed U2, U3, U5, U6, U7: MCP6L01Rx-xOT, Package_TO_SOT_SMD:SOT-23-5, symbol Amplifier_Operational:MCP6L01Rx-xOT
- added D4: S5971, OptoDevice:Osram_BPW34S-SMD, symbol Sensor_Optical:BPW34-SMD
- added U2: MCP6004, symbol Amplifier_Operational:MCP6004
- added U3: OPA2381, Package_SO:SOIC-8_3.9x4.9mm_P1.27mm, symbol Amplifier_Operational:OPA2340
- added U5: CD4051B, MUX:DIP794W45P254L1969H508Q16, symbol Analog_Switch:CD4051B
- C1, C2: value C -> 1uF
- D1: value BPW34-SMD -> S5971
- D2: value IR26-21C_L110_TR8 -> MTE8120CP 805nm
- D3: value IR26-21C_L110_TR8 -> MTSM0013-844-IR 1350 nM
- R4, R5: value R -> 27R
Connections:
- net Sinal is gone; now on net GND: C2.2
- net 3v3: now also U1.3.3 (3V3), U2.4 (V+), U3.8 (V+)
- net GND: now also U1.G (GND), D4.2 (A), U2.10 (+), U2.11 (V-), U2.12 (+), U2.3 (+), U2.5 (+), U3.3 (+), U3.4 (V-), U3.5 (+)
- net LED1: no longer U1.8 (GPIO8)
- net LED2: no longer U1.9 (GPIO9)
- net at C1.1, D1.1 (K): now also U3.2 (-); no longer C2.1
- net IN_AD: now reaches U1.0 (GPIO0)
- net IN_AD: now also U5.3 (X)
- net BIT_0: now reaches U1.7 (GPIO7)
- net BIT_0: now also U5.11 (A)
- new net: C2.1, D4.1 (K), U3.6 (-)
- new net BIT_1: U1.8 (GPIO8), U5.10 (B)
- new net OUTLED1: U2.2 (-), U2.6 (-)
- new net OUTLED2: U2.13 (-), U2.9 (-)
- new net OUT_AC_LED1: U2.7, U5.2 (X6)
- new net OUT_AC_LED2: U2.14, U5.1 (X4)
- new net OUT_DC_LED1: U2.1, U5.4 (X7)
- new net OUT_DC_LED2: U2.8, U5.5 (X5)
- new net OUT_LED1: U3.1
- new net OUT_LED2: U3.7
- no-connect marks 0 -> 5
Other:
- note added: "RNCF1206TKW27R0"
- moved on the sheet: C1, C3, C4, D1, D2, D3, R4, R5, U1, U4

Commit message: V2
Parts:
- added U6: CD4051B, MUX:DIP794W45P254L1969H508Q16, symbol Analog_Switch:CD4051B
Connections:
- net 3v3: now also U5.16 (VDD)
- net GND: now also U5.6 (INH), U5.7 (VEE), U5.8 (VSS)
- net LED1: now also U1.1 (GPIO1)
- net LED2: now also U1.2 (GPIO2)
- net OUT_AC_LED1: now also U5.15 (X2); no longer U5.2 (X6)
- net OUT_AC_LED2: now also U5.13 (X0); no longer U5.1 (X4)
- net OUT_DC_LED1: now also U5.12 (X3); no longer U5.4 (X7)
- net OUT_DC_LED2: now also U5.14 (X1); no longer U5.5 (X5)
- no-connect marks 5 -> 1
Other:
- moved on the sheet: U1

Commit message: ORGANIZEI
Parts:
- removed U6: CD4051B, MUX:DIP794W45P254L1969H508Q16, symbol Analog_Switch:CD4051B
- added C5: 0.1uF, Capacitor_SMD:C_0603_1608Metric_Pad1.08x0.95mm_HandSolder, symbol Device:C
- added R1, R2, R3, R4: R, symbol Device:R
- added U7: LTC6910-1CTS8PBF, LTC6910-1CTS8PBF:SOT65P280X100-8N, symbol LTC6910-1CTS8PBF:LTC6910-1CTS8PBF
Connections:
- net 3v3: now also C5.1, U7.8 (V+)
- net GND: now also C5.2, U7.2 (AGND), U7.4 (V-)
- net IN_AD: no longer U5.3 (X)
- net OUT_LED1: now also R4.2
- net OUT_LED2: now also R2.2
- net at C2.1, D4.1 (K): now also R1.2; no longer U3.6 (-)
- net at C1.1, D1.1 (K): now also R3.2; no longer U3.2 (-)
- net LTC_B0: now reaches U1.4 (GPIO4)
- net LTC_B0: now also U7.5 (G0)
- net LTC_B1: now reaches U1.5 (GPIO5)
- net LTC_B1: now also U7.6 (G1)
- net LTC_B2: now reaches U1.6 (GPIO6)
- net LTC_B2: now also U7.7 (G2)
- new net: R3.1, R4.1, U3.2 (-)
- new net: R1.1, R2.1, U3.6 (-)
- new net OUT_ADC: U7.1 (OUT)
- new net SAÍDA SEM GANHO: U5.3 (X), U7.3 (IN)
Other:
- note added: "AMPLIFICADOR DE TRANSIMPEDÂNCIA"
- note added: "CAPTURA DE SINAL"
- note added: "CONTROLADOR"
- note added: "GANHO PROGRAMÁVEL"
- note added: "MUX PARA SELECIONAR O SINAL"
- note added: "PASSA BAIXA"
- note added: "PASSA FAIXA"
- note added: "REGULADOR DE TENSÃO"
- moved on the sheet: C1, C2, C3, C4, D1, D2, D3, D4, R4, R5, U2A, U2B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

Commit message: Atualização da placa
Parts:
- removed D1: S5971, OptoDevice:Osram_BPW34S-SMD, symbol Sensor_Optical:BPW34-SMD
- removed R4: 27R, Resistor_SMD:R_0603_1608Metric_Pad0.98x0.95mm_HandSolder, symbol Device:R
- removed R4: R, symbol Device:R
- removed U2: MCP6004, symbol Amplifier_Operational:MCP6004
- removed U3: OPA2381, Package_SO:SOIC-8_3.9x4.9mm_P1.27mm, symbol Amplifier_Operational:OPA2340
- removed U5: CD4051B, MUX:DIP794W45P254L1969H508Q16, symbol Analog_Switch:CD4051B
- added C6, C7, C8: C, symbol Device:C
- added D1: MTE8120CP 805nm, LED_SMD:LED_1206_3216Metric, symbol LED:IR26-21C_L110_TR8
- added Q1, Q2: BC337, Package_TO_SOT_THT:TO-92_Inline, symbol Transistor_BJT:BC337
- added R4, R6, R7, R8, R9: R, symbol Device:R
- added U3: MCP6002-xMC, Package_DFN_QFN:DFN-8-1EP_3x2mm_P0.5mm_EP1.75x1.45mm, symbol Amplifier_Operational:MCP6002-xMC
- added U6: MCP601R, Package_TO_SOT_SMD:SOT-23-5, symbol Amplifier_Operational:MCP601R
- C1: value 1uF -> C; footprint Capacitor_SMD:C_0603_1608Metric_Pad1.08x0.95mm_HandSolder -> (none)
- R5: value 27R -> R; footprint Resistor_SMD:R_0603_1608Metric_Pad0.98x0.95mm_HandSolder -> (none)
Connections:
- net BIT_1 is gone; now on net LED1: U1.8 (GPIO8)
- net OUT_ADC is gone; now on net Estágio3_Filtro: U7.1 (OUT)
- net SAÍDA SEM GANHO is gone; now on net Estágio 2_Ganho: U7.3 (IN)
- net 3v3: now also D2.2 (A), D1.2 (A), U3.8 (V+), U6.5 (V+)
- net GND: now also Q1.3 (E), Q2.3 (E), R7.1, U3.2 (-), U3.4 (V-), U3.5 (+), U3.9 (V-), U6.2 (V-), U6.3 (+); no longer D2.1 (K), D3.1 (K)
- net LED1: now also R4.1; no longer U1.1 (GPIO1)
- net LED2: now also U1.9 (GPIO9); no longer U1.2 (GPIO2)
- net LTC_B0: now also U1.10 (GPIO10); no longer U1.4 (GPIO4)
- net LTC_B1: now also U1.20 (GPIO20); no longer U1.5 (GPIO5)
- net LTC_B2: now also U1.21 (GPIO21); no longer U1.6 (GPIO6)
- net at C2.1, D4.1 (K): now also R2.1, U6.4 (-); no longer R1.2
- net at R3.1: now also R1.2, C6.1
- net at C1.1, R3.2: now also U3.3 (+)
- net at D3.2 (A): no longer R5.2
- net Estágio3_Filtro: now reaches R1.1
- net Estágio3_Filtro: no longer R2.1
- net BIT_0: no longer names the net of U1.7 (GPIO7)
- net IN_AD renamed PB - entrada AD
- net PB - entrada AD: now also C6.2, C8.1, U3.1
- net OUT_LED2 renamed Estágio 2_Ganho
- net Estágio 2_Ganho: now also U6.1
- new net: D1.1 (K), R8.2
- new net: Q1.1 (C), R8.1
- new net: Q1.2 (B), R4.2
- new net: Q2.1 (C), R9.1
- new net: D2.1 (K), R9.2
- new net: C7.1, C8.2, R6.1
- new net: Q2.2 (B), R5.2
- new net: C7.2, R7.2, U3.6 (-)
- new net PF - entrada AD: R6.2, U1.5 (GPIO5), U3.7
- no-connect marks 1 -> 6
Other:
- note added: "1"
- note added: "2"
- note added: "3"
- note added: "PASSA ALTA"
- note removed: "MUX PARA SELECIONAR O SINAL"
- note removed: "PASSA FAIXA"
- note removed: "RNCF1206TKW27R0"
- moved on the sheet: C2, C3, C4, D2, D3, D4, R2, U1, U4

Commit message: inicio pcb
Parts:
- C1, C6, C7, C8: footprint (none) -> Capacitor_SMD:C_0603_1608Metric_Pad1.08x0.95mm_HandSolder
- R1, R2, R3, R4, R5, R6, R7, R8, R9: footprint (none) -> Resistor_SMD:R_0603_1608Metric
Changed lines of the file:
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@@
 			)
 		)
-		(property "Footprint" ""
+		(property "Footprint" "Resistor_SMD:R_0603_1608Metric"
 			(at 271.018 144.78 90)
 			(effects
@@
 			)
 		)
-		(property "Footprint" ""
+		(property "Footprint" "Resistor_SMD:R_0603_1608Metric"
 			(at 146.05 23.368 90)
 			(effects
@@
 			)
 		)
-		(property "Footprint" ""
+		(property "Footprint" "Resistor_SMD:R_0603_1608Metric"
 			(at 62.23 51.308 90)
 			(effects
@@
 			)
 		)
-		(property "Footprint" ""
+		(property "Footprint" "Resistor_SMD:R_0603_1608Metric"
 			(at 41.91 33.528 90)
 			(effects
@@
 			)
 		)
-		(property "Footprint" ""
+		(property "Footprint" "Resistor_SMD:R_0603_1608Metric"
 			(at 212.09 155.448 90)
 			(effects
@@
 			)
 		)
-		(property "Footprint" ""
+		(property "Footprint" "Capacitor_SMD:C_0603_1608Metric_Pad1.08x0.95mm_HandSolder"
 			(at 76.2 19.3548 0)
 			(effects
@@
 			)
 		)
-		(property "Footprint" ""
+		(property "Footprint" "Capacitor_SMD:C_0603_1608Metric_Pad1.08x0.95mm_HandSolder"
 			(at 63.1952 39.37 0)
 			(effects
@@
 			)
 		)
-		(property "Footprint" ""
+		(property "Footprint" "Resistor_SMD:R_0603_1608Metric"
 			(at 226.568 144.78 90)
 			(effects
@@
 			)
 		)
-		(property "Footprint" ""
+		(property "Footprint" "Capacitor_SMD:C_0603_1608Metric_Pad1.08x0.95mm_HandSolder"
 			(at 53.34 57.4548 0)
 			(effects
@@
 			)
 		)
-		(property "Footprint" ""
+		(property "Footprint" "Resistor_SMD:R_0603_1608Metric"
 			(at 56.388 63.5 90)
 			(effects
@@
 			)
 		)
-		(property "Footprint" ""
+		(property "Footprint" "Resistor_SMD:R_0603_1608Metric"
 			(at 55.88 33.528 90)
 			(effects
@@
 			)
 		)
-		(property "Footprint" ""
+		(property "Footprint" "Capacitor_SMD:C_0603_1608Metric_Pad1.08x0.95mm_HandSolder"
 			(at 44.45 57.4548 0)
 			(effects
@@
 			)
 		)
-		(property "Footprint" ""
+		(property "Footprint" "Resistor_SMD:R_0603_1608Metric"
 			(at 257.81 155.448 90)
 			(effects
