File: Elétrica/glicosimetro/glicosimetro.kicad_pcb (KiCad board)
At the start: 2 copper layers, 96.2 x 67.5 mm, 20 parts, among them U1 ESP32-C3_SUPERMINI, U2 MCP6L01Rx-xOT, U3 MCP6L01Rx-xOT, U4 LM1117DT-3.3, U5 MCP6L01Rx-xOT, U6 MCP6L01Rx-xOT, U7 MCP6L01Rx-xOT

Commit message: inicio pcb
Parts:
- removed the D3 at (192.4, 113.3)
- removed the D3 at (192.4, 85.9)
- removed U2, U5: MCP6L01Rx-xOT, Package_TO_SOT_SMD:SOT-23-5
- added C5: 0.1uF, Capacitor_SMD:C_0603_1608Metric_Pad1.08x0.95mm_HandSolder, F.Cu at (147.7, 118.6)
- added C6: C, Capacitor_SMD:C_0603_1608Metric_Pad1.08x0.95mm_HandSolder, F.Cu at (180.8, 126.9)
- added C7: C, Capacitor_SMD:C_0603_1608Metric_Pad1.08x0.95mm_HandSolder, F.Cu at (180.8, 129.4)
- added C8: C, Capacitor_SMD:C_0603_1608Metric_Pad1.08x0.95mm_HandSolder, F.Cu at (180.8, 131.9)
- added D3: MTSM0013-844-IR 1350 nM, LED_SMD:LED_1206_3216Metric, F.Cu at (185.8, 128.2)
- added D4: S5971, OptoDevice:Osram_BPW34S-SMD, F.Cu at (158.5, 91.5)
- added Q1: BC337, Package_TO_SOT_THT:TO-92_Inline, F.Cu at (169.3, 85.8)
- added Q2: BC337, Package_TO_SOT_THT:TO-92_Inline, F.Cu at (163.7, 101.9)
- added R6: R, Resistor_SMD:R_0603_1608Metric, F.Cu at (168.9, 128.9)
- added R7: R, Resistor_SMD:R_0603_1608Metric, F.Cu at (168.9, 131.4)
- added R8: R, Resistor_SMD:R_0603_1608Metric, F.Cu at (168.9, 133.9)
- added R9: R, Resistor_SMD:R_0603_1608Metric, F.Cu at (168.9, 136.4)
- C2: value C -> 1uF
- D1: value BPW34-SMD -> MTE8120CP 805nm; footprint OptoDevice:Osram_BPW34S-SMD -> LED_SMD:LED_1206_3216Metric
- D2: value IR26-21C_L110_TR8 -> MTE8120CP 805nm
- R1, R2, R3, R4, R5: footprint Resistor_SMD:R_0603_1608Metric_Pad0.98x0.95mm_HandSolder -> Resistor_SMD:R_0603_1608Metric
- U3: value MCP6L01Rx-xOT -> MCP6002-xMC; footprint Package_TO_SOT_SMD:SOT-23-5 -> Package_DFN_QFN:DFN-8-1EP_3x2mm_P0.5mm_EP1.75x1.45mm
- U6: value MCP6L01Rx-xOT -> MCP601R
- U7: value MCP6L01Rx-xOT -> LTC6910-1CTS8PBF; footprint Package_TO_SOT_SMD:SOT-23-5 -> LTC6910-1CTS8PBF:SOT65P280X100-8N
- moved D1 58.4 mm to (141.9, 117.9)
- moved C2 55.2 mm to (147.7, 116.1)
- moved R5 49.2 mm to (168.9, 126.4), turned to 0 degrees
- moved R4 45.7 mm to (168.9, 123.9), turned to 0 degrees
- moved U6 45.4 mm to (148.1, 112.6)
- moved U3 45.2 mm to (152.8, 116.8)
- moved C3 44.8 mm to (174.8, 126.1)
- moved C4 44.8 mm to (174.8, 131.9)
- moved U7 40.0 mm to (153.0, 112.2)
- moved C1 38.2 mm to (180.8, 124.4)
- moved R1 35.7 mm to (168.9, 116.3)
- moved R2 35.7 mm to (168.9, 118.9)
- moved R3 35.7 mm to (168.9, 121.4)
- moved U4 28.1 mm to (177.8, 119.1)
- moved D2 25.5 mm to (185.8, 124.9)
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Connections:
- C1 pad 1: Net-(D1-K) -> Net-(U3A-+)
- C2 pad 1: Net-(D1-K) -> Net-(D4-K)
- C2 pad 2: Sinal -> GND
- D1 pad 2: GND -> 3v3
- D2 pad 1: GND -> Net-(D2-K)
- D2 pad 2: Net-(D2-A) -> 3v3
- R1 pad 1: Net-(D1-K) -> Estágio3_Filtro
- R1 pad 2: Sinal -> Net-(C6-Pad1)
- R2 pad 1: GND -> Net-(D4-K)
- R2 pad 2: Net-(R2-Pad2) -> Estágio 2_Ganho
- R3 pad 1: Net-(R2-Pad2) -> Net-(C6-Pad1)
- R3 pad 2: 3v3 -> Net-(U3A-+)
- R4 pad 2: Net-(D2-A) -> Net-(Q1-B)
- U1 pad 0: unconnected-(U1-GPIO0-Pad0) -> PB - entrada AD
- U1 pad 10: unconnected-(U1-GPIO10-Pad10) -> LTC_B0
- U1 pad 20: unconnected-(U1-GPIO20-Pad20) -> LTC_B1
- U1 pad 21: unconnected-(U1-GPIO21-Pad21) -> LTC_B2
- U1 pad 3.3: unconnected-(U1-3V3-Pad3.3) -> 3v3
- U1 pad 5: unconnected-(U1-GPIO5-Pad5) -> PF - entrada AD
- U1 pad G: unconnected-(U1-GND-PadG) -> GND
- U3 pad 1: Sinal -> PB - entrada AD
- U3 pad 2: 3V3 -> GND
- U3 pad 3: REF -> Net-(U3A-+)
- U3 pad 4: Net-(D1-K) -> GND
- U6 pad 1: unconnected-(U6-Pad1) -> Estágio 2_Ganho
- U6 pad 2: unconnected-(U6-V+-Pad2) -> GND
- U6 pad 3: unconnected-(U6-+-Pad3) -> GND
- U6 pad 4: unconnected-(U6---Pad4) -> Net-(D4-K)
- U6 pad 5: unconnected-(U6-V--Pad5) -> 3v3
- U7 pad 1: unconnected-(U7-Pad1) -> Estágio3_Filtro
- U7 pad 2: unconnected-(U7-V+-Pad2) -> GND
- U7 pad 3: unconnected-(U7-+-Pad3) -> Estágio 2_Ganho
- U7 pad 4: unconnected-(U7---Pad4) -> GND
- U7 pad 5: unconnected-(U7-V--Pad5) -> LTC_B0

Commit message: Simulação
Parts:
- moved R1 44.3 mm to (206.2, 92.5)
- moved C3 39.9 mm to (203.3, 98.1)
- moved C4 39.9 mm to (203.3, 104.0)
- moved D2 39.9 mm to (214.4, 96.9)
- moved D3 39.9 mm to (214.4, 100.3)
- moved U4 39.9 mm to (206.3, 91.2)
- moved C6 39.9 mm to (209.3, 99.0)
- moved R9 39.9 mm to (197.4, 108.5)
- moved C1 39.9 mm to (209.3, 96.5)
- moved C7 39.9 mm to (209.3, 101.5)
- moved R2 39.9 mm to (197.4, 90.9)
- moved R3 39.9 mm to (197.4, 93.4)
- moved R4 39.9 mm to (197.4, 95.9)
- moved R5 39.9 mm to (197.4, 98.4)
- moved R6 39.9 mm to (197.4, 100.9)
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Other:
- board size 96.2 x 67.5 mm -> 96.5 x 46.1 mm
